File: B200-GPSDO.sch (EAGLE design)
At the start: 17 parts, among them U1 LEA-6T, U2 NC7SZ125, U3 NC7SZ125, U4 GPSDO

Commit message: update
Parts:
- U2, U3: value NC7SZ125 -> NC7SZ125M5X
Changed lines of the file:
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@@
 <part name="GND6" library="supply1" deviceset="GND" device=""/>
 <part name="GND7" library="supply1" deviceset="GND" device=""/>
-<part name="U2" library="B200-GPSDO" deviceset="NC7SZ125" device=""/>
-<part name="U3" library="B200-GPSDO" deviceset="NC7SZ125" device=""/>
+<part name="U2" library="B200-GPSDO" deviceset="NC7SZ125" device="" value="NC7SZ125M5X"/>
+<part name="U3" library="B200-GPSDO" deviceset="NC7SZ125" device="" value="NC7SZ125M5X"/>
 <part name="GND8" library="supply1" deviceset="GND" device=""/>
 <part name="R1" library="rcl" deviceset="R-US_" device="R0805" value="1k"/>
